File: Geckonator.sch (KiCad schematic (older format))
At the start: 15 parts, among them P1 USART0, P2 DEBUG, P3 USB_A, P4 CONN_01X02, P5 CONN_02X03, U1 EFM32HG309

Commit message: Added PDF schematic, licensing info and updated to KiCad 5.0
Signed-off-by: Thomas Flummer <tf@flummer.net>
Parts:
- C1, C2, C3: symbol C_Small -> device:C_Small
- D1, D2: symbol LED -> Geckonator-rescue:LED
- P1, P2: symbol CONN_01X04 -> Geckonator-rescue:CONN_01X04
- P3: symbol USB_A -> Geckonator-rescue:USB_A
- P4: symbol CONN_01X02 -> Geckonator-rescue:CONN_01X02
- P5: symbol CONN_02X03 -> Geckonator-rescue:CONN_02X03
- R1, R2, R3, R4: symbol R_Small -> device:R_Small
- U1: symbol EFM32HG309 -> efm32hg309:EFM32HG309
Changed lines of the file:
@@
-EESchema Schematic File Version 2
-LIBS:power
-LIBS:device
-LIBS:transistors
-LIBS:conn
-LIBS:linear
-LIBS:regul
-LIBS:74xx
-LIBS:cmos4000
-LIBS:adc-dac
-LIBS:memory
-LIBS:xilinx
-LIBS:microcontrollers
-LIBS:dsp
-LIBS:microchip
-LIBS:analog_switches
-LIBS:motorola
-LIBS:texas
-LIBS:intel
-LIBS:audio
-LIBS:interface
-LIBS:digital-audio
-LIBS:philips
-LIBS:display
-LIBS:cypress
-LIBS:siliconi
-LIBS:opto
-LIBS:atmel
-LIBS:contrib
-LIBS:valves
-LIBS:efm32hg309
+EESchema Schematic File Version 4
 LIBS:Geckonator-cache
-EELAYER 25 0
+EELAYER 26 0
 EELAYER END
 $Descr A4 11693 8268
@@
 Date "$Id$"
 Rev ""
-Comp "hackmeister.dk"
-Comment1 "License: CC-BY-SA"
+Comp "https://geckonator.dk"
+Comment1 "License: Creative Commons Attribution-ShareAlike 4.0 International License (CC BY-SA 4.0)"
 Comment2 ""
 Comment3 ""
@@
 $EndDescr
 $Comp
-L C_Small C2
+L device:C_Small C2
 U 1 1 5798B89B
 P 6125 3975
@@
 $EndComp
 $Comp
-L GND #PWR01
+L power:GND #PWR01
 U 1 1 5798BA02
 P 6200 4175
@@
 $EndComp
 $Comp
-L C_Small C3
+L device:C_Small C3
 U 1 1 5798BA32
 P 7000 3850
@@
 $EndComp
 $Comp
-L C_Small C1
+L device:C_Small C1
 U 1 1 5798BCD7
 P 5725 4025
@@
 USB_5V
 $Comp
-L R_Small R3
+L device:R_Small R3
 U 1 1 5798C3BC
 P 5650 3100
@@
 $EndComp
 $Comp
-L R_Small R4
+L device:R_Small R4
 U 1 1 5798C529
 P 5650 3175
@@
 $EndComp
 $Comp
-L CONN_01X04 P2
+L Geckonator-rescue:CONN_01X04 P2
 U 1 1 5798E965
 P 2450 3925
@@
 DBG_SWDIO
 $Comp
-L GND #PWR02
+L power:GND #PWR02
 U 1 1 5798EEB6
 P 2700 4125
@@
 $EndComp
 $Comp
-L +3V3 #PWR03
+L power:+3V3 #PWR03
 U 1 1 5798EF1D
 P 6000 3575
@@
 $EndComp
 $Comp
-L +3V3 #PWR04
+L power:+3V3 #PWR04
 U 1 1 5798F04E
 P 2700 3725
@@
 $EndComp
 $Comp
-L LED D1
+L Geckonator-rescue:LED D1
 U 1 1 5798F0D5
 P 3325 2425
@@
 $EndComp
 $Comp
-L LED D2
+L Geckonator-rescue:LED D2
 U 1 1 5798F173
 P 3550 2425
@@
 $EndComp
 $Comp
-L R_Small R2
+L device:R_Small R2
 U 1 1 5798F38A
 P 3825 2175
@@
 $EndComp
 $Comp
-L R_Small R1
+L device:R_Small R1
 U 1 1 5798F3FD
 P 3825 2025
@@
 $EndComp
 $Comp
-L CONN_01X04 P1
+L Geckonator-rescue:CONN_01X04 P1
 U 1 1 5798FD61
 P 2100 3125
@@
 $EndComp
 $Comp
-L GND #PWR05
+L power:GND #PWR05
 U 1 1 5798FD6B
 P 2350 3325
@@
 $EndComp
 $Comp
-L +3V3 #PWR06
+L power:+3V3 #PWR06
 U 1 1 5798FD73
 P 2350 2925
@@
 RUSB_D+
 $Comp
-L +3V3 #PWR07
+L power:+3V3 #PWR07
 U 1 1 579B6568
 P 3450 2675
@@
 $EndComp
 $Comp
-L EFM32HG309 U1
+L efm32hg309:EFM32HG309 U1
 U 1 1 5798B6D7
 P 4400 4175
@@
 $EndComp
 Wire Wire Line
-	5500 3350 6125 3350
+	5500 3350 5750 3350
 Wire Wire Line
 	5750 3625 5500 3625
@@
 Connection ~ 6125 4125
 Wire Wire Line
-	6125 3350 6125 3875
-Wire Wire Line
-	5750 3350 5750 3925
+	6125 3350 6125 3625
+Wire Wire Line
+	5750 3350 5750 3625
 Wire Wire Line
 	5550 3100 5500 3100
@@
 	5500 3175 5550 3175
 Wire Wire Line
-	5500 3025 6350 3025
+	5500 3025 6300 3025
 Wire Wire Line
 	5750 3100 6200 3100
@@
 	6200 3175 5750 3175
 Wire Wire Line
-	5500 4125 7000 4125
+	5500 4125 5950 4125
 Wire Wire Line
 	7000 4125 7000 3950
@@
 	3450 2675 3450 2625
 Wire Wire Line
-	3325 2625 3550 2625
+	3325 2625 3450 2625
 Connection ~ 3450 2625
 Wire Wire Line
@@
 	4100 3125 4200 3125
 $Comp
-L GND #PWR08
+L power:GND #PWR08
 U 1 1 57A1602A
 P 4030 4035
@@
 	4030 4025 4030 4035
 $Comp
-L USB_A P3
+L Geckonator-rescue:USB_A P3
 U 1 1 587A59FD
 P 6650 3225
@@
 $EndComp
 $Comp
-L CONN_01X02 P4
+L Geckonator-rescue:CONN_01X02 P4
 U 1 1 587A9872
 P 4400 4450
@@
 $EndComp
 $Comp
-L GND #PWR09
+L power:GND #PWR09
 U 1 1 587A9986
 P 4025 4600
@@
 	3225 3075 2300 3075
 $Comp
-L CONN_02X03 P5
+L Geckonator-rescue:CONN_02X03 P5
 U 1 1 587AAF85
 P 3225 4900
@@
 PE12
 $Comp
-L GND #PWR?
+L power:GND #PWR?
 U 1 1 587AA2E1
 P 6750 3625
@@
 Wire Wire Line
 	6750 3525 6750 3625
+Wire Wire Line
+	5750 3350 6125 3350
+Wire Wire Line
+	5750 3625 5750 3700
+Wire Wire Line
+	6200 4125 6350 4125
+Wire Wire Line
+	6125 4125 6200 4125
+Wire Wire Line
+	6300 3025 6350 3025
+Wire Wire Line
+	5750 3700 5750 3775
+Wire Wire Line
+	5750 3775 5750 3850
+Wire Wire Line
+	5750 3850 5750 3925
+Wire Wire Line
+	5950 4125 6125 4125
+Wire Wire Line
+	6125 3625 6125 3875
+Wire Wire Line
+	6350 4125 7000 4125
+Wire Wire Line
+	3450 2625 3550 2625
 $EndSCHEMATC
